Commit message: Update mid360.xacro configuration

File: urdf/mid360.xacro (robot description, xacro)
@@ -8,4 +8,7 @@
   <xacro:property name="noise_mean" value="0.0"/>
   <xacro:property name="noise_stddev" value="0.01"/>
+  <xacro:property name="imu_update_rate" value="100"/>
+  <xacro:property name="gyro_noise_stddev" value="2e-4"/>
+  <xacro:property name="accel_noise_stddev" value="1.7e-2"/>
   <xacro:property name="mass" value="0.4" />
   <xacro:property name="length" value="0.1" />
@@ -14,18 +17,18 @@
   <xacro:macro name="box_inertia" params="m w h d">
     <inertial>
-      <origin xyz="0 0 0" rpy="${pi/2} 0 ${pi/2}"/>
+      <origin xyz="0 0 0" rpy="${M_PI/2} 0 ${M_PI/2}"/>
       <mass value="${m}"/>
       <inertia ixx="${(m/12) * (h*h + d*d)}" ixy="0.0" ixz="0.0" iyy="${(m/12) * (w*w + d*d)}" iyz="0.0" izz="${(m/12) * (w*w + h*h)}"/>
     </inertial>
   </xacro:macro>
-  <xacro:macro name="mid360" params="name:='' parent:= 'base_link' topic:='mid360' *origin ">
-<link name="${name}">
-<xacro:box_inertia m="${length}" w="${width}" d="${length}" h="${height}"/>
-  <visual>
+  <xacro:macro name="mid360" params="name:='' parent:= 'base_link' topic:='mid360' imu_topic:='imu/data' *origin ">
+    <link name="${name}">
+      <xacro:box_inertia m="${length}" w="${width}" d="${length}" h="${height}"/>
+      <visual>
         <geometry>
             <box size="${length} ${width} ${height}"/>
         </geometry>
-  </visual>
-</link>
+      </visual>
+    </link>
     <joint name="${name}_joint" type="fixed">
       <parent link="${parent}"/>
@@ -34,44 +37,67 @@
     </joint>
     <gazebo reference="${name}">
-      <sensor type="ray" name="${name}">
+      <sensor type="ray" name="${name}_lidar">
         <pose>0 0 0 0 0 0</pose>
         <visualize>true</visualize>
-        <update_rate>10</update_rate>
-        <!-- This ray plgin is only for visualization. -->
+        <update_rate>4</update_rate>
         <plugin name="${name}_plugin" filename="libros2_livox.so">
-			<ray>
-			  <scan>
-				<horizontal>
-				<samples>100</samples>
-				<resolution>1</resolution>
-				<min_angle>${0}</min_angle>
-				<max_angle>${2*M_PI}</max_angle>
-				</horizontal>
-				<vertical>
-				<samples>360</samples>
-				<resolution>1</resolution>
-				<min_angle>${-7.22/180*M_PI}</min_angle>
-				<max_angle>${55.22/180*M_PI}</max_angle>
-				</vertical>
-			  </scan>
-			  <range>
-				<min>${laser_min_range}</min>
-				<max>${laser_max_range}</max>
-				<resolution>${resolution}</resolution>
-			  </range>
-			  <noise>
-				<type>gaussian</type>
-				<mean>${noise_mean}</mean>
-				<stddev>${noise_stddev}</stddev>
-			  </noise>
-			</ray>
+          <ray>
+            <scan>
+              <horizontal>
+                <samples>100</samples>
+                <resolution>1</resolution>
+                <min_angle>${0}</min_angle>
+                <max_angle>${2*M_PI}</max_angle>
+              </horizontal>
+              <vertical>
+                <samples>360</samples>
+                <resolution>1</resolution>
+                <min_angle>${-7.22/180*M_PI}</min_angle>
+                <max_angle>${55.22/180*M_PI}</max_angle>
+              </vertical>
+            </scan>
+            <range>
+              <min>${laser_min_range}</min>
+              <max>${laser_max_range}</max>
+              <resolution>${resolution}</resolution>
+            </range>
+            <noise>
+              <type>gaussian</type>
+              <mean>${noise_mean}</mean>
+              <stddev>${noise_stddev}</stddev>
+            </noise>
+          </ray>
           <visualize>false</visualize>
-		  <samples>${samples}</samples>
-		  <downsample>1</downsample>
-		  <csv_file_name>$(find ros2_livox_simulation)/scan_mode/mid360.csv</csv_file_name>
-		  <topic>${topic}</topic>
+          <samples>${samples}</samples>
+          <downsample>1</downsample>
+          <csv_file_name>$(find ros2_livox_simulation)/scan_mode/mid360.csv</csv_file_name>
+          <topic>${topic}</topic>
         </plugin>
       </sensor>
-    </gazebo>
+      <sensor name="${name}_imu" type="imu">
+        <pose>0 0 0 0 0 0</pose> <always_on>true</always_on>
+        <update_rate>${imu_update_rate}</update_rate>
+        <visualize>false</visualize>
+        <plugin name="${name}_imu_plugin" filename="libgazebo_ros_imu_sensor.so">
+          <ros>
+            <namespace>/</namespace>
+            <output_type>sensor_msgs/msg/Imu</output_type>
+            <topic_name>${imu_topic}</topic_name> <frame_id>${name}</frame_id>
+          </ros>
+          <imu>
+            <angular_velocity>
+              <x><noise type="gaussian"><mean>0.0</mean><stddev>${gyro_noise_stddev}</stddev></noise></x>
+              <y><noise type="gaussian"><mean>0.0</mean><stddev>${gyro_noise_stddev}</stddev></noise></y>
+              <z><noise type="gaussian"><mean>0.0</mean><stddev>${gyro_noise_stddev}</stddev></noise></z>
+            </angular_velocity>
+            <linear_acceleration>
+              <x><noise type="gaussian"><mean>0.0</mean><stddev>${accel_noise_stddev}</stddev></noise></x>
+              <y><noise type="gaussian"><mean>0.0</mean><stddev>${accel_noise_stddev}</stddev></noise></y>
+              <z><noise type="gaussian"><mean>0.0</mean><stddev>${accel_noise_stddev}</stddev></noise></z>
+            </linear_acceleration>
+          </imu>
+        </plugin>
+        </sensor>
+      </gazebo>
   </xacro:macro>
 </robot>
